File: 4_layer.kicad_sch (KiCad schematic)
At the start: 51 parts, among them J1 Conn_01x05_Pin, Q1 BSC265N10LSFG, Q2 BSC265N10LSFG, Q3 BSC265N10LSFG, Q4 BSC265N10LSFG, Q5 BSC265N10LSFG, Q6 BSC265N10LSFG, SW1 SW_Push, SW2 SW_Nidec_CAS-120A1, U1 ADP2108AUJ-3.3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

Commit message: Add files via upload
Connections:
- net PH_A: no longer R10.2, R2.2, R5.1
- net PH_B: no longer R3.2, R6.1, R9.2
- net PH_C: no longer R4.2, R7.1, R8.2
- net HSE: no longer names the net of C12.2, U2.5 (PF0), X1.2
- net HSE: no longer C13.2, U2.6 (PF1), X1.1
- new net: R3.2, R6.1, R9.2
- new net: R10.2, R2.2, R5.1
- new net: R4.2, R7.1, R8.2
- new net: C13.2, U2.6 (PF1), X1.1
Changed lines of the file:
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@@
-		)
-	)
-	(label "HSE"
-		(at 214.63 72.39 0)
-		(fields_autoplaced yes)
-		(effects
-			(font
-				(size 1.27 1.27)
-			)
-			(justify left bottom)
-		)
-	)
-	(label "PH_B"
-		(at 180.34 115.57 0)
-		(fields_autoplaced yes)
-		(effects
-			(font
-				(size 1.27 1.27)
-			)
-			(justify left bottom)
 		)
 	)
 	(label "BOOT0_SW"
 		(at 208.28 54.61 0)
-		(fields_autoplaced yes)
-		(effects
-			(font
-				(size 1.27 1.27)
-			)
-			(justify left bottom)
-		)
-	)
-	(label "PH_A"
-		(at 182.88 118.11 0)
 		(fields_autoplaced yes)
 		(effects
@@
 		)
 	)
-	(label "HSE"
-		(at 213.36 64.77 0)
-		(fields_autoplaced yes)
-		(effects
-			(font
-				(size 1.27 1.27)
-			)
-			(justify left bottom)
-		)
-	)
 	(label "BOOT0"
 		(at 218.44 57.15 0)
 		(fields_autoplaced yes)
 		(effects
-			(font
-				(size 1.27 1.27)
-			)
-			(justify left bottom)
-		)
-	)
-	(label "PH_C"
-		(at 177.8 118.11 0)
-		(fields_autoplaced yes)
-		(effects
