File: 4_layer.kicad_pcb (KiCad board)
At the start: 4 copper layers, 37.2 x 34.2 mm, 54 parts, among them J1 Conn_01x05_Pin, Q1 BSC265N10LSFG, Q2 BSC265N10LSFG, Q3 BSC265N10LSFG, Q4 BSC265N10LSFG, Q5 BSC265N10LSFG, Q6 BSC265N10LSFG, SW1 SW_Push, SW2 SW_Nidec_CAS-120A1, U1 ADP2108AUJ-3.3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

Commit message: Add files via upload
Parts:
- removed ? (x3): , 
- moved J1 32.4 mm to (189.2, 57.5)
- moved R1 3.67 mm to (184.8, 52.2), turned to 0 degrees
- moved C12 1.08 mm to (195.4, 58.5)
- moved C13 1.08 mm to (200.7, 58.5)
- moved C15 1.00 mm to (180.0, 38.5)
- moved C19 1.00 mm to (204.4, 38.5)
- moved U3 0.98 mm to (184.3, 37.9)
- moved C14 0.97 mm to (186.3, 41.2)
- moved C18 0.96 mm to (210.8, 41.2)
- moved U5 0.95 mm to (208.8, 37.9)
- moved C16 0.88 mm to (198.5, 41.2)
- moved C8 0.86 mm to (206.0, 45.0), turned to 0 degrees
- moved C17 0.82 mm to (192.2, 38.5)
- moved BAT_+1 0.79 mm to (179.2, 52.0)
- moved BAT_-1 0.79 mm to (179.2, 44.0)
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Connections:
- C12 pad 2: /HSE -> Net-(U2-PF0)
- C13 pad 2: /HSE -> Net-(U2-PF1)
- R10 pad 2: PH_A -> Net-(R10-Pad2)
- R2 pad 2: PH_A -> Net-(R10-Pad2)
- R3 pad 2: PH_B -> Net-(R3-Pad2)
- R4 pad 2: PH_C -> Net-(R4-Pad2)
- R5 pad 1: PH_A -> Net-(R10-Pad2)
- R6 pad 1: PH_B -> Net-(R3-Pad2)
- R7 pad 1: PH_C -> Net-(R4-Pad2)
- R8 pad 2: PH_C -> Net-(R4-Pad2)
- R9 pad 2: PH_B -> Net-(R3-Pad2)
- U2 pad 5: /HSE -> Net-(U2-PF0)
- U2 pad 6: /HSE -> Net-(U2-PF1)
- X1 pad 1: /HSE -> Net-(U2-PF1)
- X1 pad 2: /HSE -> Net-(U2-PF0)
Routing:
- net +3.3V: track 0.00 -> 93.4 mm, vias 0 -> 3
- net PH_A: track 3.86 -> 48.5 mm, vias 0 -> 9
- net PH_B: track 2.38 -> 37.5 mm, vias 0 -> 9
- net SW_JT_RESET: track 0.00 -> 31.9 mm, vias 0 -> 1
- net PH_C: track 2.41 -> 32.9 mm, vias 0 -> 9
- net SWDIO: track 0.00 -> 27.4 mm, vias 0 -> 1
- net +3.3VA: track 0.00 -> 25.1 mm, vias 0 -> 2
- net GND: track 0.00 -> 23.7 mm, vias 0 -> 16
- net AL: track 0.00 -> 20.1 mm, vias 0 -> 2
- net Net-(Q3-G): track 0.00 -> 18.7 mm
- net Net-(Q1-G): track 0.00 -> 18.6 mm
- net COMP1_INM: track 0.00 -> 18.4 mm, vias 0 -> 2
- net Net-(Q4-G): track 0.00 -> 18.2 mm
- net BH: track 0.00 -> 15.8 mm, vias 0 -> 2
- net CH: track 0.00 -> 14.8 mm
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- added copper zone on B.Cu, net GND
- added copper zone on F.Cu, net GND
- added copper zone on In1.Cu, net GND
- added copper zone on In2.Cu, net GND
- added copper zone on In2.Cu, net PH_A
- added copper zone on In2.Cu, net PH_B
- added copper zone on In2.Cu, net PH_C
Other:
- board size 37.2 x 34.2 mm -> 37.6 x 35 mm
- board text added: "A"
- board text added: "B"
- board text added: "C"

Commit message: Add files via upload
Parts:
- moved C14 1.80 mm to (188.1, 41.2)
- moved C15 1.80 mm to (181.8, 38.4)
- moved U3 1.80 mm to (186.1, 37.8)
- moved U4 1.74 mm to (198.3, 37.8)
- moved C16 1.74 mm to (200.3, 41.2)
- moved C17 1.74 mm to (193.9, 38.4)
- moved U5 1.61 mm to (210.4, 37.7)
- moved C19 1.61 mm to (206.1, 38.4)
- moved C18 1.61 mm to (212.4, 41.1)
- moved C7 0.66 mm to (195.4, 42.4), turned to 180 degrees
- moved TP2 0.53 mm to (199.2, 26.1)
- moved TP3 0.50 mm to (211.3, 26.1)
- moved TP1 0.50 mm to (187.1, 26.1)
- moved C1 0.42 mm to (178.4, 48.6)
- moved J1 0.40 mm to (189.2, 58.0)
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Routing:
- net +15V: track 6.35 -> 58.4 mm, vias 22 -> 19
- net PH_C: track 32.9 -> 60.1 mm
- net PH_B: track 37.5 -> 62.1 mm
- net PH_A: track 48.5 -> 69.1 mm
- net +3.3V: track 93.4 -> 77.7 mm, vias 3 -> 4
- net SW_JT_RESET: track 31.9 -> 21.9 mm, vias 1 -> 2
- net SWDIO: track 27.4 -> 23.2 mm, vias 1 -> 2
- net Net-(Q1-G): track 18.6 -> 15.3 mm, vias 0 -> 2
- net +3.3VA: track 25.1 -> 22.2 mm
- net CL: track 10.5 -> 13.4 mm
- net AL: track 20.1 -> 17.4 mm
- net Net-(Q4-G): track 18.2 -> 20.0 mm
- net Net-(Q5-G): track 7.71 -> 5.95 mm
- net SWCLK: track 12.0 -> 13.7 mm, vias 0 -> 2
- net Net-(Q6-G): track 7.65 -> 6.00 mm
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Other:
- board size 37.6 x 35 mm -> 37.9 x 35 mm
